Commit message: gmapping works

File: defs/pioneer3at.xacro (robot description, xacro)
@@ -33,4 +33,11 @@
 		<material value="Gazebo/Red"/>
 	</gazebo>
+<link name="odom">
+</link>
+<joint name="odom_base" type="fixed">
+		<origin xyz="0 0 0" rpy="0 0 0"/>
+		<parent link="odom"/>
+		<child link="base_link"/>
+	</joint>
 <!-- Top -->
 	<link name="top_plate">
@@ -358,5 +365,5 @@
     <commandTopic>cmd_vel</commandTopic>
     <odometryTopic>odom</odometryTopic>
-    <odometryFrame>base_link</odometryFrame>
+    <odometryFrame>odom</odometryFrame>
   </plugin>
 </gazebo>

Commit message: fixed Odometry frame and broadcastTF

File: defs/pioneer3at.xacro (robot description, xacro)
@@ -33,11 +33,19 @@
 		<material value="Gazebo/Red"/>
 	</gazebo>
-<link name="odom">
+<!--link name="odom">
 </link>
-<joint name="odom_base" type="fixed">
+<joint name="odom_base" type="floating">
 		<origin xyz="0 0 0" rpy="0 0 0"/>
 		<parent link="odom"/>
 		<child link="base_link"/>
-	</joint>
+	</joint-->
+<!--<link name="map">
+</link-->
+<!--<joint name="map_odom" type="fixed">
+		<origin xyz="0 0 0" rpy="0 0 0"/>
+		<parent link="map"/>
+		<child link="odom"/>
+	</joint>
+	-->
 <!-- Top -->
 	<link name="top_plate">
@@ -353,5 +361,5 @@
 <gazebo>
   <plugin name="skid_steer_drive_controller" filename="libgazebo_ros_skid_steer_drive.so">
-    <updateRate>100.0</updateRate>
+    <updateRate>50000.0</updateRate>
     <robotNamespace>/</robotNamespace>
     <leftFrontJoint>p3at_front_left_wheel_joint</leftFrontJoint>
@@ -366,4 +374,5 @@
     <odometryTopic>odom</odometryTopic>
     <odometryFrame>odom</odometryFrame>
+    <broadcastTF>1</broadcastTF>
   </plugin>
 </gazebo>
